Commit message: Vertical Pick and Place working

File: src/arm_urdf/urdf/ArmPlate.xacro (robot description, xacro)
@@ -895,4 +895,11 @@
         </collision>
     </link>
+    <link name="grasp_frame">
+    </link>
+    <joint name="grasp_to_hand" type= "fixed">
+    <origin xyz="-0.015 -0.06 -0.17" rpy="0.0 0.0 -0.35" />
+    <parent link="gcomp1" />
+    <child link="grasp_frame" />
+    </joint>
     <joint name="base_to_robot" type="fixed">
     <origin xyz="0.0 0.35 -0.07" rpy="1.57 0.0 0.0" />
@@ -950,4 +957,5 @@
         <child link="Spur_Gear_driven" />
         <axis xyz="-0.9470809999999998 -0.024682999999999993 -0.320045" />
+          <limit lower="-1000" upper="1000" effort="10" velocity="10"/>
     </joint>
     <joint name="Spur_Gear_driven_Rigid_64" type="fixed">
@@ -1050,4 +1058,5 @@
         <child link="Spur_Gear_motor" />
         <axis xyz="-0.947081 0.32004499999999997 -0.024683000000000014" />
+        <limit lower="-1000" upper="1000" effort="10" velocity="10"/>
     </joint>
     <joint name="Base_link_Rigid_91" type="fixed">

Commit message: Resolved Soft finger issue and planner issue, changed mtc code to use pre defined place pose

File: src/arm_urdf/urdf/ArmPlate.xacro (robot description, xacro)
@@ -1059,4 +1059,5 @@
         <axis xyz="-0.947081 0.32004499999999997 -0.024683000000000014" />
         <limit lower="-1000" upper="1000" effort="10" velocity="10"/>
+        <mimic joint="gcomp1_Revolute_63" multiplier="-1.0" offset="0"/>
     </joint>
     <joint name="Base_link_Rigid_91" type="fixed">

File: src/arm_urdf_moveit_config/config/ArmPlate.ros2_control.xacro (robot description, xacro)
@@ -57,5 +57,5 @@
                 <state_interface name="velocity"/>
             </joint>
-            <joint name="AX_12A_04_4_Revolute_90">
+            <!-- <joint name="AX_12A_04_4_Revolute_90">
                 <command_interface name="position"/>
                 <state_interface name="position">
@@ -63,5 +63,5 @@
                 </state_interface>
                 <state_interface name="velocity"/>
-            </joint>
+            </joint> -->
         </ros2_control>
     </xacro:macro>

Commit message: Added joint and velocity limits. Fixed start and known states. Using CHOMP optimizer on TRRT

File: src/arm_urdf/urdf/ArmPlate.xacro (robot description, xacro)
@@ -974,15 +974,17 @@
         <child link="STEPPER_MOTOR" />
     </joint>
-    <joint name="STEPPER_MOTOR_Revolute_74" type="continuous">
+    <joint name="STEPPER_MOTOR_Revolute_74" type="revolute">
         <origin xyz="0.02167662 0.0 0.01609733" rpy="-1.5707963267948966 -1.859084879483064e-17 -2.795186720719627e-17" />
         <parent link="STEPPER_MOTOR" />
         <child link="link23" />
         <axis xyz="-0.802838 0.596197 -4.6143341949499234e-17" />
-    </joint>
-    <joint name="AX_12A_04_3_Revolute_75" type="continuous">
+        <limit lower="-1.74533" upper="1.74533" effort="1.0" velocity="0.25" />
+    </joint>
+    <joint name="AX_12A_04_3_Revolute_75" type="revolute">
         <origin xyz="0.0003050900000000034 -0.00041084000000000124 0.006379510000000011" rpy="3.141592653589793 -8.798523825835593e-34 1.6320449438997825e-16" />
         <parent link="AX_12A_04_3" />
         <child link="Component20" />
         <axis xyz="-0.047670999999999984 -0.06419400000000001 0.996798" />
+         <limit lower="-3.14159" upper="3.14159" effort="1.0" velocity="0.25" />
     </joint>
     <joint name="AX_12A_03_1_Rigid_76" type="fixed">
@@ -1006,9 +1008,10 @@
         <child link="AX_12A_03_1" />
     </joint>
-    <joint name="AX_12A_04_1_Revolute_80" type="continuous">
+    <joint name="AX_12A_04_1_Revolute_80" type="revolute">
         <origin xyz="0.006061319999999988 0.0020482900000000017 -0.00015796999999992067" rpy="3.141592653589793 -8.868773770931429e-17 -3.0769740127124206e-34" />
         <parent link="AX_12A_04_1" />
         <child link="Component1_1" />
         <axis xyz="-0.947081 0.320045 -0.024682999999999983" />
+        <limit lower="-1.970796" upper="1.170796" effort="1.0" velocity="0.25" />
     </joint>
     <joint name="Component1_1_Rigid_81" type="fixed">
@@ -1037,9 +1040,10 @@
         <child link="AX_12A_03_2" />
     </joint>
-    <joint name="AX_12A_04_2_Revolute_86" type="continuous">
+    <joint name="AX_12A_04_2_Revolute_86" type="revolute">
         <origin xyz="-0.0007006800000000269 0.0025238100000000065 0.005839470000000091" rpy="-3.141592653589793 -1.0408340855860838e-17 -5.204170427930417e-18" />
         <parent link="AX_12A_04_2" />
         <child link="gcomp1" />
         <axis xyz="0.10948099999999998 0.39434500000000017 0.9124180000000002" />
+        <limit lower="-3.14159" upper="3.14159" effort="1.0" velocity="0.25" />
     </joint>
     <joint name="Base_link_Rigid_87" type="fixed">
@@ -1076,9 +1080,10 @@
         <child link="Universal_hub" />
     </joint>
-    <joint name="Nema_34_v3_Revolute_94" type="continuous">
+    <joint name="Nema_34_v3_Revolute_94" type="revolute">
         <origin xyz="-0.03500000000000004 -0.007828609999999998 -0.0481634" rpy="3.141592653589793 -1.5707963267948966 0" />
         <parent link="Nema_34_v3" />
         <child link="Component7" />
         <axis xyz="-0.802838 -0.596197 4.456646163201019e-17" />
+        <limit lower="-1.396263" upper="1.396263" effort="1.0" velocity="0.25" />
     </joint>
     <joint name="Component7_Rigid_95" type="fixed">
@@ -1092,9 +1097,10 @@
         <child link="Component6" />
     </joint>
-    <joint name="firstDOF_final_Revolute_100" type="continuous">
+    <joint name="firstDOF_final_Revolute_100" type="revolute">
         <origin xyz="-0.284 0.07999999999999999 -0.135" rpy="6.310887241768095e-30 -4.930380657631324e-32 -3.111507638930571e-61" />
         <parent link="firstDOF_final" />
         <child link="Base_link" />
         <axis xyz="0.0 -1.0 -3.1554436208840472e-30" />
+        <limit lower="-3.14159" upper="3.14159" effort="1.0" velocity="0.25" />
     </joint>
     <joint name="Wheel_motor_2_Revolute_105" type="continuous">

Commit message: Interfaced with Gazebo

File: src/arm_urdf/urdf/ArmPlate.xacro (robot description, xacro)
@@ -2,4 +2,9 @@
 <robot name="ArmPlate">
     <link name="base_footprint"/>
+    <link name="world"/>
+    <joint name="base_to_world" type="fixed">
+    <parent link ="world"/>
+    <child link = "base_footprint"/>
+    </joint>
     <link name="AX_12A_04_4">
         <inertial>
@@ -1063,5 +1068,4 @@
         <axis xyz="-0.947081 0.32004499999999997 -0.024683000000000014" />
         <limit lower="-1000" upper="1000" effort="10" velocity="10"/>
-        <mimic joint="gcomp1_Revolute_63" multiplier="-1.0" offset="0"/>
     </joint>
     <joint name="Base_link_Rigid_91" type="fixed">

File: src/arm_urdf_moveit_config/config/ArmPlate.ros2_control.xacro (robot description, xacro)
@@ -3,8 +3,13 @@
     <xacro:macro name="ArmPlate_ros2_control" params="name initial_positions_file">
         <xacro:property name="initial_positions" value="${load_yaml(initial_positions_file)['initial_positions']}"/>
-        <ros2_control name="${name}" type="system">
+      <gazebo>
+        <plugin name="gazebo_ros2_control" filename="libgazebo_ros2_control.so">
+            <parameters>$(find arm_urdf_moveit_config)/config/ros2_controllers.yaml</parameters>
+        </plugin>
+      </gazebo>
+        <ros2_control name="GazeboSimSystem" type="system">
             <hardware>
                 <!-- By default, set up controllers for simulation. This won't work on real hardware -->
-                <plugin>mock_components/GenericSystem</plugin>
+                <plugin>gazebo_ros2_control/GazeboSystem</plugin>
             </hardware>
             <joint name="firstDOF_final_Revolute_100">
@@ -57,5 +62,5 @@
                 <state_interface name="velocity"/>
             </joint>
-            <!-- <joint name="AX_12A_04_4_Revolute_90">
+            <joint name="AX_12A_04_4_Revolute_90">
                 <command_interface name="position"/>
                 <state_interface name="position">
@@ -63,5 +68,5 @@
                 </state_interface>
                 <state_interface name="velocity"/>
-            </joint> -->
+            </joint>
         </ros2_control>
     </xacro:macro>

Commit message: Teleoped diff drive controller

File: src/arm_urdf/urdf/ArmPlate.xacro (robot description, xacro)
@@ -2,4 +2,9 @@
 <robot name="ArmPlate">
     <link name="base_footprint"/>
+    <!-- <link name="world"/>
+    <joint name="base_to_world" type="floating">
+    <parent link ="world"/>
+    <child link = "base_footprint"/>
+    </joint> -->
     <link name="AX_12A_04_4">
         <inertial>
@@ -1063,5 +1068,5 @@
         <axis xyz="-0.947081 0.32004499999999997 -0.024683000000000014" />
         <limit lower="-1000" upper="1000" effort="10" velocity="10"/>
-        <mimic joint="gcomp1_Revolute_63" multiplier="-1.0" offset="0"/>
+        <!-- <mimic joint="gcomp1_Revolute_63" multiplier="-1.0" offset="0"/> -->
     </joint>
     <joint name="Base_link_Rigid_91" type="fixed">
@@ -1109,4 +1114,5 @@
         <child link="Component53" />
         <axis xyz="1.0 2.635647389719074e-60 2.139937261679685e-14" />
+        <dynamics damping="1.0" friction="1.0"/>
     </joint>
     <joint name="Wheel_motor_4_Revolute_106" type="continuous">
@@ -1115,4 +1121,5 @@
         <child link="Component54" />
         <axis xyz="-1.0 8.586479331114432e-60 -2.1399372616796854e-14" />
+        <dynamics damping="1.0" friction="1.0"/>
     </joint>
     <joint name="Wheel_motor_1_Revolute_107" type="continuous">
@@ -1121,4 +1128,5 @@
         <child link="Component55" />
         <axis xyz="-1.0 -7.16708135826507e-61 -2.139937261679685e-14" />
+        <dynamics damping="1.0" friction="1.0"/>
     </joint>
     <joint name="Wheel_motor_3_Revolute_108" type="continuous">
@@ -1127,4 +1135,5 @@
         <child link="Component56" />
         <axis xyz="1.0 -8.619515182870853e-61 2.139937261679685e-14" />
+        <dynamics damping="1.0" friction="1.0"/>
     </joint>
     <joint name="base_final-v3_Rigid_114" type="fixed">

File: src/arm_urdf_moveit_config/config/ArmPlate.ros2_control.xacro (robot description, xacro)
@@ -3,8 +3,13 @@
     <xacro:macro name="ArmPlate_ros2_control" params="name initial_positions_file">
         <xacro:property name="initial_positions" value="${load_yaml(initial_positions_file)['initial_positions']}"/>
+      <gazebo>
+        <plugin name="gazebo_ros2_control" filename="libgazebo_ros2_control.so">
+            <parameters>$(find arm_urdf_moveit_config)/config/ros2_controllers.yaml</parameters>
+        </plugin>
+      </gazebo>
         <ros2_control name="${name}" type="system">
             <hardware>
                 <!-- By default, set up controllers for simulation. This won't work on real hardware -->
-                <plugin>mock_components/GenericSystem</plugin>
+                <plugin>gazebo_ros2_control/GazeboSystem</plugin>
             </hardware>
             <joint name="firstDOF_final_Revolute_100">
@@ -57,5 +62,25 @@
                 <state_interface name="velocity"/>
             </joint>
-            <!-- <joint name="AX_12A_04_4_Revolute_90">
+            <joint name="Wheel_motor_2_Revolute_105">
+              <command_interface name="velocity"/>
+              <state_interface name="velocity"/>
+              <state_interface name="position"/>
+            </joint>
+            <joint name="Wheel_motor_1_Revolute_107">
+              <command_interface name="velocity"/>
+              <state_interface name="velocity"/>
+              <state_interface name="position"/>
+            </joint>
+            <joint name="Wheel_motor_3_Revolute_108">
+              <command_interface name="velocity"/>
+              <state_interface name="velocity"/>
+              <state_interface name="position"/>
+            </joint>
+            <joint name="Wheel_motor_4_Revolute_106">
+              <command_interface name="velocity"/>
+              <state_interface name="velocity"/>
+              <state_interface name="position"/>
+            </joint>
+            <joint name="AX_12A_04_4_Revolute_90">
                 <command_interface name="position"/>
                 <state_interface name="position">
@@ -63,5 +88,5 @@
                 </state_interface>
                 <state_interface name="velocity"/>
-            </joint> -->
+            </joint>
         </ros2_control>
     </xacro:macro>

Commit message: shifted back

File: src/arm_urdf/urdf/ArmPlate.xacro (robot description, xacro)
@@ -1109,31 +1109,27 @@
         <limit lower="-3.14159" upper="3.14159" effort="1.0" velocity="0.25" />
     </joint>
-    <joint name="Wheel_motor_2_Revolute_105" type="continuous">
+    <joint name="Wheel_motor_2_Revolute_105" type="fixed">
         <origin xyz="-1.7763568394002505e-17 0.0 0.026999999999999993" rpy="-1.5707963267948966 1.5707963267948948 0" />
         <parent link="Wheel_motor_2" />
         <child link="Component53" />
         <axis xyz="1.0 2.635647389719074e-60 2.139937261679685e-14" />
-        <dynamics damping="1.0" friction="1.0"/>
-    </joint>
-    <joint name="Wheel_motor_4_Revolute_106" type="continuous">
+    </joint>
+    <joint name="Wheel_motor_4_Revolute_106" type="fixed">
         <origin xyz="-1.7763568394002505e-17 -3.552713678800501e-17 0.026999999999999993" rpy="1.5707963267948966 -1.570796326794895 0" />
         <parent link="Wheel_motor_4" />
         <child link="Component54" />
         <axis xyz="-1.0 8.586479331114432e-60 -2.1399372616796854e-14" />
-        <dynamics damping="1.0" friction="1.0"/>
-    </joint>
-    <joint name="Wheel_motor_1_Revolute_107" type="continuous">
+    </joint>
+    <joint name="Wheel_motor_1_Revolute_107" type="fixed">
         <origin xyz="-0.0020000000000000287 0.0056568599999999945 0.026999999999999993" rpy="1.5707963267948966 -1.570796326794895 0" />
         <parent link="Wheel_motor_1" />
         <child link="Component55" />
         <axis xyz="-1.0 -7.16708135826507e-61 -2.139937261679685e-14" />
-        <dynamics damping="1.0" friction="1.0"/>
-    </joint>
-    <joint name="Wheel_motor_3_Revolute_108" type="continuous">
+    </joint>
+    <joint name="Wheel_motor_3_Revolute_108" type="fixed">
         <origin xyz="-1.7763568394002505e-17 0.005999999999999961 0.026999999999999993" rpy="-1.5707963267948966 1.5707963267948948 0" />
         <parent link="Wheel_motor_3" />
         <child link="Component56" />
         <axis xyz="1.0 -8.619515182870853e-61 2.139937261679685e-14" />
-        <dynamics damping="1.0" friction="1.0"/>
     </joint>
     <joint name="base_final-v3_Rigid_114" type="fixed">

File: src/arm_urdf_moveit_config/config/ArmPlate.ros2_control.xacro (robot description, xacro)
@@ -3,13 +3,13 @@
     <xacro:macro name="ArmPlate_ros2_control" params="name initial_positions_file">
         <xacro:property name="initial_positions" value="${load_yaml(initial_positions_file)['initial_positions']}"/>
-      <gazebo>
+      <!-- <gazebo>
         <plugin name="gazebo_ros2_control" filename="libgazebo_ros2_control.so">
             <parameters>$(find arm_urdf_moveit_config)/config/ros2_controllers.yaml</parameters>
         </plugin>
-      </gazebo>
+      </gazebo> -->
         <ros2_control name="${name}" type="system">
             <hardware>
                 <!-- By default, set up controllers for simulation. This won't work on real hardware -->
-                <plugin>gazebo_ros2_control/GazeboSystem</plugin>
+              <plugin>mock_components/GenericSystem</plugin>
             </hardware>
             <joint name="firstDOF_final_Revolute_100">
@@ -62,5 +62,5 @@
                 <state_interface name="velocity"/>
             </joint>
-            <joint name="Wheel_motor_2_Revolute_105">
+            <!-- <joint name="Wheel_motor_2_Revolute_105">
               <command_interface name="velocity"/>
               <state_interface name="velocity"/>
@@ -81,9 +81,8 @@
               <state_interface name="velocity"/>
               <state_interface name="position"/>
-            </joint>
+            </joint> -->
             <joint name="AX_12A_04_4_Revolute_90">
                 <command_interface name="position"/>
                 <state_interface name="position">
-                  <param name="initial_value">${initial_positions['AX_12A_04_4_Revolute_90']}</param>
                 </state_interface>
                 <state_interface name="velocity"/>

Commit message: Tried fixing world frame issue

File: src/arm_urdf/urdf/ArmPlate.xacro (robot description, xacro)
@@ -2,9 +2,9 @@
 <robot name="ArmPlate">
     <link name="base_footprint"/>
-    <!-- <link name="world"/>
+    <link name="world"/>
     <joint name="base_to_world" type="floating">
     <parent link ="world"/>
     <child link = "base_footprint"/>
-    </joint> -->
+    </joint>
     <link name="AX_12A_04_4">
         <inertial>
